File: hardware/logic/logic.brd (EAGLE design)
At the start: 41.6 x 34.2 mm, 30 parts, among them U1 STM32F103CBT6, X1 22-23-2021

Commit message: fixes in logic board. now support 6 channels. add debug
Parts:
- added C4: 100uf, Seeed-Capacitor:AVX-B
- renumbered U$1 to R3, U$10 to R11, U$3 to R4, U$4 to R5, U$5 to R6, U$6 to R7, U$7 to R8, U$8 to R9, U$9 to R10
Connections:
- net GND: now also C4.+
- net V3.3: now also C4.-
Routing:
- net V3.3: track 136.4 -> 147.5 mm, vias 4 -> 5

Commit message: logic version 2.2
Connections:
- net USART1_RX: no longer X1.2
- net USART1_TX: now also X1.2
Routing:
- net GND: track 157.8 -> 114.7 mm, vias 4 -> 3
- net FAN_CTRL: track 22.8 -> 58.6 mm, vias 1 -> 4
- net USART1_TX: track 23.5 -> 44.6 mm, vias 1 -> 0
- net V3.3: track 147.5 -> 130.6 mm, vias 5 -> 6
- net ZONE1: track 37.8 -> 21.4 mm
- net I2C1_SDA: track 72.4 -> 84.4 mm, vias 3 -> 2
- net USART1_RX: track 28.8 -> 17.7 mm
- net ZONE5: track 41.2 -> 35.4 mm, vias 3 -> 1
- net ZONE3: track 24.7 -> 19.3 mm, vias 1 -> 2
- net ZONE4: track 93.4 -> 89.4 mm, vias 4 -> 2
- net ZONE6: track 35.2 -> 31.8 mm, vias 1 -> 2
- net SWDCLK: track 21.7 -> 21.0 mm, vias 0 -> 1
- net SWDIO: track 14.5 -> 15.0 mm
- removed copper zone on layer 16, net GND
Other:
- board text added: "WF Logic v2.2"
- board text removed: "WF Logic v2.1"
