File: hardware/logic/logic.sch (EAGLE design)
At the start: 30 parts, among them U1 STM32F103CBT6, X1 22-23-2021

Commit message: fixes in logic board. now support 6 channels. add debug
Parts:
- added C4: 100uf, Seeed-Capacitor:TANTALUM-SMD-100UF-10V(AVX-B)
- renumbered U$1 to R3, U$10 to R11, U$3 to R4, U$4 to R5, U$5 to R6, U$6 to R7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
Connections:
- net GND: now also C4.+
- net V3.3: now also C4.-

Commit message: logic version 2.2
Connections:
- net USART1_RX: no longer X1-2.S
- net USART1_TX: now also X1-2.S
